File: cryptostick.sch (KiCad schematic (older format))
At the start: 24 parts, among them J1 SIM_JACKET, J2 USB_A, P1 CONN_4, U1 STM32F103TB, U2 CAT6217-330, U3 NUF2221W1, X1 12MHz

Commit message: Changed boot0 jumper to THT. Decreased VDD via size.
Parts:
- removed R4: 0, ~, symbol R
- added JP1: JUMPER, ~, symbol JUMPER
- renumbered R5 to R4
Connections:
- net +3.3V: now also JP1.2
- net BOOT0: now also JP1.1
Changed lines of the file:
@@
 LIBS:stf202
 LIBS:power
-LIBS:device
-LIBS:conn
 LIBS:sst25vf032b
 LIBS:cryptostick-cache
+LIBS:w_analog
+LIBS:w_connectors
+LIBS:w_device
+LIBS:w_logic
+LIBS:w_memory
+LIBS:w_microcontrollers
+LIBS:w_opto
+LIBS:w_relay
+LIBS:w_rtx
+LIBS:w_transistor
+LIBS:w_vacuum
 LIBS:cryptostick-cache
 EELAYER 27 0
@@
 Sheet 1 1
 Title ""
-Date "25 feb 2014"
+Date "2 mar 2014"
 Rev ""
 Comp ""
@@
 $EndComp
 $Comp
-L GND #PWR01
+L GND #PWR7
 U 1 1 500508DE
 P 2750 1250
-F 0 "#PWR01" H 2750 1250 30  0001 C CNN
+F 0 "#PWR7" H 2750 1250 30  0001 C CNN
 F 1 "GND" H 2750 1180 30  0001 C CNN
 F 2 "" H 2750 1250 60  0001 C CNN
@@
 $EndComp
 $Comp
-L GND #PWR02
+L GND #PWR1
 U 1 1 5005072E
 P 1600 1700
-F 0 "#PWR02" H 1600 1700 30  0001 C CNN
+F 0 "#PWR1" H 1600 1700 30  0001 C CNN
 F 1 "GND" H 1600 1630 30  0001 C CNN
 F 2 "" H 1600 1700 60  0001 C CNN
@@
 $EndComp
 $Comp
-L GND #PWR03
+L GND #PWR11
 U 1 1 4F801E27
 P 4400 7150
-F 0 "#PWR03" H 4400 7150 30  0001 C CNN
+F 0 "#PWR11" H 4400 7150 30  0001 C CNN
 F 1 "GND" H 4400 7080 30  0001 C CNN
 F 2 "" H 4400 7150 60  0001 C CNN
@@
 $EndComp
 $Comp
-L GND #PWR04
+L GND #PWR14
 U 1 1 4F4EDF5A
 P 5150 1950
-F 0 "#PWR04" H 5150 1950 30  0001 C CNN
+F 0 "#PWR14" H 5150 1950 30  0001 C CNN
 F 1 "GND" H 5150 1880 30  0001 C CNN
 F 2 "" H 5150 1950 60  0001 C CNN
@@
 $EndComp
 $Comp
-L +3,3V #PWR05
+L +3,3V #PWR12
 U 1 1 4F4EDE58
 P 4850 1500
-F 0 "#PWR05" H 4850 1460 30  0001 C CNN
+F 0 "#PWR12" H 4850 1460 30  0001 C CNN
 F 1 "+3,3V" H 4850 1610 30  0000 C CNN
 F 2 "" H 4850 1500 60  0001 C CNN
@@
 $EndComp
 $Comp
-L GND #PWR06
+L GND #PWR4
 U 1 1 4E82CDD0
 P 1850 3600
-F 0 "#PWR06" H 1850 3600 30  0001 C CNN
+F 0 "#PWR4" H 1850 3600 30  0001 C CNN
 F 1 "GND" H 1850 3530 30  0001 C CNN
 F 2 "" H 1850 3600 60  0001 C CNN
@@
 $EndComp
 $Comp
-L GND #PWR07
+L GND #PWR13
 U 1 1 4E2D76FE
 P 4850 6100
-F 0 "#PWR07" H 4850 6100 30  0001 C CNN
+F 0 "#PWR13" H 4850 6100 30  0001 C CNN
 F 1 "GND" H 4850 6030 30  0001 C CNN
 F 2 "" H 4850 6100 60  0001 C CNN
@@
 $EndComp
 $Comp
-L GND #PWR08
+L GND #PWR15
 U 1 1 4E2D6DF1
 P 5300 6400
-F 0 "#PWR08" H 5300 6400 30  0001 C CNN
+F 0 "#PWR15" H 5300 6400 30  0001 C CNN
 F 1 "GND" H 5300 6330 30  0001 C CNN
 F 2 "" H 5300 6400 60  0001 C CNN
@@
 $EndComp
 $Comp
-L GND #PWR09
+L GND #PWR5
 U 1 1 4E2D6A81
 P 2600 4700
-F 0 "#PWR09" H 2600 4700 30  0001 C CNN
+F 0 "#PWR5" H 2600 4700 30  0001 C CNN
 F 1 "GND" H 2600 4630 30  0001 C CNN
 F 2 "" H 2600 4700 60  0001 C CNN
@@
 $EndComp
 $Comp
-L +3,3V #PWR010
+L +3,3V #PWR17
 U 1 1 4E2D6574
 P 5850 4500
-F 0 "#PWR010" H 5850 4460 30  0001 C CNN
+F 0 "#PWR17" H 5850 4460 30  0001 C CNN
 F 1 "+3,3V" H 5850 4610 30  0000 C CNN
 F 2 "" H 5850 4500 60  0001 C CNN
@@
 $EndComp
 $Comp
-L GND #PWR011
+L GND #PWR18
 U 1 1 4E2D6572
 P 5850 5100
-F 0 "#PWR011" H 5850 5100 30  0001 C CNN
+F 0 "#PWR18" H 5850 5100 30  0001 C CNN
 F 1 "GND" H 5850 5030 30  0001 C CNN
 F 2 "" H 5850 5100 60  0001 C CNN
@@
 $EndComp
 $Comp
-L +3,3V #PWR012
+L +3,3V #PWR6
 U 1 1 4E2D63FA
 P 2700 4050
-F 0 "#PWR012" H 2700 4010 30  0001 C CNN
+F 0 "#PWR6" H 2700 4010 30  0001 C CNN
 F 1 "+3,3V" H 2700 4160 30  0000 C CNN
 F 2 "" H 2700 4050 60  0001 C CNN
@@
 $EndComp
 $Comp
-L GND #PWR013
+L GND #PWR9
 U 1 1 4E2D63F8
 P 3100 3800
-F 0 "#PWR013" H 3100 3800 30  0001 C CNN
+F 0 "#PWR9" H 3100 3800 30  0001 C CNN
 F 1 "GND" H 3100 3730 30  0001 C CNN
 F 2 "" H 3100 3800 60  0001 C CNN
@@
 $EndComp
 $Comp
-L +3,3V #PWR014
+L +3,3V #PWR10
 U 1 1 4E2D167C
 P 3350 3050
-F 0 "#PWR014" H 3350 3010 30  0001 C CNN
+F 0 "#PWR10" H 3350 3010 30  0001 C CNN
 F 1 "+3,3V" H 3350 3160 30  0000 C CNN
 F 2 "" H 3350 3050 60  0001 C CNN
@@
 $EndComp
 $Comp
-L GND #PWR015
+L GND #PWR8
 U 1 1 4E2D167A
 P 2850 3200
-F 0 "#PWR015" H 2850 3200 30  0001 C CNN
+F 0 "#PWR8" H 2850 3200 30  0001 C CNN
 F 1 "GND" H 2850 3130 30  0001 C CNN
 F 2 "" H 2850 3200 60  0001 C CNN
@@
 $EndComp
 $Comp
-L GND #PWR016
+L GND #PWR20
 U 1 1 4E2D1452
 P 6450 3300
-F 0 "#PWR016" H 6450 3300 30  0001 C CNN
+F 0 "#PWR20" H 6450 3300 30  0001 C CNN
 F 1 "GND" H 6450 3230 30  0001 C CNN
 F 2 "" H 6450 3300 60  0001 C CNN
@@
 $EndComp
 $Comp
-L +3,3V #PWR017
+L +3,3V #PWR16
 U 1 1 4E2D124C
 P 5850 3050
-F 0 "#PWR017" H 5850 3010 30  0001 C CNN
+F 0 "#PWR16" H 5850 3010 30  0001 C CNN
 F 1 "+3,3V" H 5850 3160 30  0000 C CNN
 F 2 "" H 5850 3050 60  0001 C CNN
@@
 $EndComp
 $Comp
-L GND #PWR018
+L GND #PWR26
 U 1 1 4E2CDAFB
 P 7350 2950
-F 0 "#PWR018" H 7350 2950 30  0001 C CNN
+F 0 "#PWR26" H 7350 2950 30  0001 C CNN
 F 1 "GND" H 7350 2880 30  0001 C CNN
 F 2 "" H 7350 2950 60  0001 C CNN
@@
 $EndComp
 $Comp
-L +3,3V #PWR019
+L +3,3V #PWR19
 U 1 1 4E2CD995
 P 6450 1300
-F 0 "#PWR019" H 6450 1260 30  0001 C CNN
+F 0 "#PWR19" H 6450 1260 30  0001 C CNN
 F 1 "+3,3V" H 6450 1410 30  0000 C CNN
 F 2 "" H 6450 1300 60  0001 C CNN
@@
 $EndComp
 $Comp
-L GND #PWR020
+L GND #PWR21
 U 1 1 4E2CD951
 P 6600 1850
-F 0 "#PWR020" H 6600 1850 30  0001 C CNN
+F 0 "#PWR21" H 6600 1850 30  0001 C CNN
 F 1 "GND" H 6600 1780 30  0001 C CNN
 F 2 "" H 6600 1850 60  0001 C CNN
@@
 $EndComp
 $Comp
-L GND #PWR021
+L GND #PWR27
 U 1 1 4E2CD945
 P 7550 1550
-F 0 "#PWR021" H 7550 1550 30  0001 C CNN
+F 0 "#PWR27" H 7550 1550 30  0001 C CNN
 F 1 "GND" H 7550 1480 30  0001 C CNN
 F 2 "" H 7550 1550 60  0001 C CNN
@@
 $EndComp
 $Comp
-L GND #PWR022
+L GND #PWR22
 U 1 1 4E2CD8F1
 P 7050 2650
-F 0 "#PWR022" H 7050 2650 30  0001 C CNN
+F 0 "#PWR22" H 7050 2650 30  0001 C CNN
 F 1 "GND" H 7050 2580 30  0001 C CNN
 F 2 "" H 7050 2650 60  0001 C CNN
@@
 $EndComp
 $Comp
-L GND #PWR023
+L GND #PWR3
 U 1 1 4E2CD35B
 P 1775 3900
-F 0 "#PWR023" H 1775 3900 30  0001 C CNN
+F 0 "#PWR3" H 1775 3900 30  0001 C CNN
 F 1 "GND" H 1775 3830 30  0001 C CNN
 F 2 "" H 1775 3900 60  0001 C CNN
@@
 $EndComp
 $Comp
-L GND #PWR024
+L GND #PWR2
 U 1 1 4E2CD351
 P 1775 3300
-F 0 "#PWR024" H 1775 3300 30  0001 C CNN
+F 0 "#PWR2" H 1775 3300 30  0001 C CNN
 F 1 "GND" H 1775 3230 30  0001 C CNN
 F 2 "" H 1775 3300 60  0001 C CNN
@@
 D-_PLUG
 $Comp
-L GND #PWR025
+L GND #PWR25
 U 1 1 4E2CCCBB
 P 7250 4150
-F 0 "#PWR025" H 7250 4150 30  0001 C CNN
+F 0 "#PWR25" H 7250 4150 30  0001 C CNN
 F 1 "GND" H 7250 4080 30  0001 C CNN
 F 2 "" H 7250 4150 60  0001 C CNN
@@
 $EndComp
 $Comp
-L GND #PWR026
+L GND #PWR28
 U 1 1 4E2CCC8D
 P 9850 4550
-F 0 "#PWR026" H 9850 4550 30  0001 C CNN
+F 0 "#PWR28" H 9850 4550 30  0001 C CNN
 F 1 "GND" H 9850 4480 30  0001 C CNN
 F 2 "" H 9850 4550 60  0001 C CNN
@@
 $Comp
 L R R4
-U 1 1 530CE600
-P 6700 5450
-F 0 "R4" V 6780 5450 40  0000 C CNN
-F 1 "0" V 6707 5451 40  0000 C CNN
-F 2 "~" V 6630 5450 30  0000 C CNN
-F 3 "~" H 6700 5450 30  0000 C CNN
-	1    6700 5450
-	0    -1   -1   0
-$EndComp
-$Comp
-L R R5
 U 1 1 530CE60F
 P 6700 5750
-F 0 "R5" V 6780 5750 40  0000 C CNN
+F 0 "R4" V 6780 5750 40  0000 C CNN
 F 1 "10k" V 6707 5751 40  0000 C CNN
 F 2 "~" V 6630 5750 30  0000 C CNN
@@
 $EndComp
 Wire Wire Line
-	6000 5450 6450 5450
+	6000 5450 6550 5450
 Wire Wire Line
 	6450 5450 6450 5750
 Wire Wire Line
-	6950 5450 7100 5450
+	6850 5450 7100 5450
 Wire Wire Line
 	6950 5750 7100 5750
@@
 	7100 5750 7100 5800
 $Comp
-L +3,3V #PWR027
+L +3,3V #PWR23
 U 1 1 530CE9AE
 P 7100 5450
-F 0 "#PWR027" H 7100 5410 30  0001 C CNN
+F 0 "#PWR23" H 7100 5410 30  0001 C CNN
 F 1 "+3,3V" H 7100 5560 30  0000 C CNN
 F 2 "" H 7100 5450 60  0000 C CNN
@@
 $EndComp
 $Comp
-L GND #PWR028
+L GND #PWR24
 U 1 1 530CE9BD
 P 7100 5800
-F 0 "#PWR028" H 7100 5800 30  0001 C CNN
+F 0 "#PWR24" H 7100 5800 30  0001 C CNN
 F 1 "GND" H 7100 5730 30  0001 C CNN
 F 2 "" H 7100 5800 60  0000 C CNN
@@
 Text Label 4950 5600 0    60   ~ 0
 BOOT1
+$Comp
+L JUMPER JP1
+U 1 1 531358A7
+P 6700 5450
+F 0 "JP1" H 6700 5600 60  0000 C CNN
+F 1 "JUMPER" H 6700 5370 40  0000 C CNN
+F 2 "~" H 6700 5450 60  0000 C CNN
+F 3 "~" H 6700 5450 60  0000 C CNN
+	1    6700 5450
+	1    0    0    -1
+$EndComp
+Connection ~ 6450 5450
 $EndSCHEMATC
