File: src/nk-start.sch (KiCad schematic (older format))
At the start: 40 parts, among them J1 SIM_JACKET, J2 USB_A, P1 CONN_4, U1 STM32F103TB, U2 CAT6217-330, U3 DF5A5.6JE, U4 MTCH101, X1 12MHz, p1 debug-pin, p2 debug-pin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

Commit message: Nitrokey Start
- SIM jack replaced with a touch button pad
Parts:
- removed C5: 0.1uF, c_0402, symbol C-RESCUE-cryptostick
- removed J1: SIM_JACKET, molex 78646-3001, symbol SIM_JACKET
- added P2: TouchPAD, TouchPad, symbol TouchPAD
- J2: symbol USB_2 -> USB_2-RESCUE-nk-start
- U1: footprint QFN36 -> QFN36_no_via
Connections:
- net at R8.2: now also U4.1 (MTI)
- net at R8.1: now also P2.1 (PIN); no longer U4.1 (MTI)
- net SCCLK: no longer names the net of U1.20 (PA8)
- net SCRST: no longer names the net of U1.30 (PB3)
- net SCSDA: no longer names the net of U1.10 (PA3)
- net SCVCC: no longer names the net of U1.31 (PB4)
- net SCVCC: no longer U1.32 (PB5)
- no-connect marks 18 -> 15
Other:
- moved on the sheet: A1, C12, C13, R10, R11, R8, R9, U4
