File: src/cryptostick.sch (KiCad schematic (older format))
At the start: 24 parts, among them J1 SIM_JACKET, J2 USB_A, P1 CONN_4, U1 STM32F103TB, U2 CAT6217-330, U3 NUF2221W1, X1 12MHz

Commit message: Pads under USB provided
USB connection exposed as pin pads, similarly how we did it at the last
hardware (FIDO U2F)
Parts:
- added W1, W2, W3, W4: TEST_1P, SMD_Packages:1Pin, symbol TEST_1P
- C1, C10, C2, C3, C4, C5, C6, C7, C8: symbol C -> C-RESCUE-cryptostick
- C11, C9: symbol CP1 -> CP1-RESCUE-cryptostick
- R1, R2, R3, R4: symbol R -> R-RESCUE-cryptostick
Changed lines of the file:
@@
 EESchema Schematic File Version 2
+LIBS:cryptostick-rescue
 LIBS:crystal-gnd
 LIBS:nuf2221w1
@@
 LIBS:stf202
 LIBS:power
+LIBS:device
+LIBS:conn
 LIBS:sst25vf032b
 LIBS:cryptostick-cache
-LIBS:w_analog
-LIBS:w_connectors
-LIBS:w_device
-LIBS:w_logic
-LIBS:w_memory
-LIBS:w_microcontrollers
-LIBS:w_opto
-LIBS:w_relay
-LIBS:w_rtx
-LIBS:w_transistor
-LIBS:w_vacuum
-LIBS:cryptostick-cache
-EELAYER 27 0
+LIBS:CONNECTOR
+LIBS:ref-packages
+EELAYER 25 0
 EELAYER END
 $Descr A4 11693 8268
@@
 	5300 6300 5300 6400
 $Comp
-L R R3
+L R-RESCUE-cryptostick R3
 U 1 1 5155A7EA
 P 5200 5850
@@
 $EndComp
 $Comp
-L GND #PWR7
+L GND-RESCUE-cryptostick #PWR7
 U 1 1 500508DE
 P 2750 1250
@@
 $EndComp
 $Comp
-L C C5
+L C-RESCUE-cryptostick C5
 U 1 1 500508D3
 P 3100 1100
@@
 $EndComp
 $Comp
-L GND #PWR1
+L GND-RESCUE-cryptostick #PWR1
 U 1 1 5005072E
 P 1600 1700
@@
 $EndComp
 $Comp
-L GND #PWR11
+L GND-RESCUE-cryptostick #PWR11
 U 1 1 4F801E27
 P 4400 7150
@@
 $EndComp
 $Comp
-L R R2
+L R-RESCUE-cryptostick R2
 U 1 1 4F801E05
 P 4700 5450
@@
 $EndComp
 $Comp
-L GND #PWR14
+L GND-RESCUE-cryptostick #PWR14
 U 1 1 4F4EDF5A
 P 5150 1950
@@
 $EndComp
 $Comp
-L GND #PWR4
+L GND-RESCUE-cryptostick #PWR4
 U 1 1 4E82CDD0
 P 1850 3600
@@
 SWCLK
 $Comp
-L CP1 C11
+L CP1-RESCUE-cryptostick C11
 U 1 1 4E2D79C8
 P 7350 2700
@@
 $EndComp
 $Comp
-L CP1 C9
+L CP1-RESCUE-cryptostick C9
 U 1 1 4E2D79BC
 P 6600 1600
@@
 $EndComp
 $Comp
-L GND #PWR13
+L GND-RESCUE-cryptostick #PWR13
 U 1 1 4E2D76FE
 P 4850 6100
@@
 $EndComp
 $Comp
-L R R1
+L R-RESCUE-cryptostick R1
 U 1 1 4E2D766E
 P 4400 5700
@@
 $EndComp
 $Comp
-L GND #PWR15
+L GND-RESCUE-cryptostick #PWR15
 U 1 1 4E2D6DF1
 P 5300 6400
@@
 $EndComp
 $Comp
-L GND #PWR5
+L GND-RESCUE-cryptostick #PWR5
 U 1 1 4E2D6A81
 P 2600 4700
@@
 $EndComp
 $Comp
-L C C3
+L C-RESCUE-cryptostick C3
 U 1 1 4E2D6A2C
 P 2600 4400
@@
 $EndComp
 $Comp
-L C C7
+L C-RESCUE-cryptostick C7
 U 1 1 4E2D6573
 P 5850 4800
@@
 $EndComp
 $Comp
-L GND #PWR18
+L GND-RESCUE-cryptostick #PWR18
 U 1 1 4E2D6572
 P 5850 5100
@@
 $EndComp
 $Comp
-L C C4
+L C-RESCUE-cryptostick C4
 U 1 1 4E2D63F9
 P 2900 3900
@@
 $EndComp
 $Comp
-L GND #PWR9
+L GND-RESCUE-cryptostick #PWR9
 U 1 1 4E2D63F8
 P 3100 3800
@@
 $EndComp
 $Comp
-L C C6
+L C-RESCUE-cryptostick C6
 U 1 1 4E2D167B
 P 3150 3100
@@
 $EndComp
 $Comp
-L GND #PWR8
+L GND-RESCUE-cryptostick #PWR8
 U 1 1 4E2D167A
 P 2850 3200
@@
 $EndComp
 $Comp
-L GND #PWR20
+L GND-RESCUE-cryptostick #PWR20
 U 1 1 4E2D1452
 P 6450 3300
@@
 $EndComp
 $Comp
-L C C8
+L C-RESCUE-cryptostick C8
 U 1 1 4E2D1296
 P 6050 3200
@@
 $EndComp
 $Comp
-L GND #PWR26
+L GND-RESCUE-cryptostick #PWR26
 U 1 1 4E2CDAFB
 P 7350 2950
@@
 $EndComp
 $Comp
-L C C10
+L C-RESCUE-cryptostick C10
 U 1 1 4E2CD9BD
 P 7350 1400
@@
 $EndComp
 $Comp
-L GND #PWR21
+L GND-RESCUE-cryptostick #PWR21
 U 1 1 4E2CD951
 P 6600 1850
@@
 $EndComp
 $Comp
-L GND #PWR27
+L GND-RESCUE-cryptostick #PWR27
 U 1 1 4E2CD945
 P 7550 1550
@@
 $EndComp
 $Comp
-L GND #PWR22
+L GND-RESCUE-cryptostick #PWR22
 U 1 1 4E2CD8F1
 P 7050 2650
@@
 $EndComp
 $Comp
-L GND #PWR3
+L GND-RESCUE-cryptostick #PWR3
 U 1 1 4E2CD35B
 P 1775 3900
@@
 $EndComp
 $Comp
-L GND #PWR2
+L GND-RESCUE-cryptostick #PWR2
 U 1 1 4E2CD351
 P 1775 3300
@@
 $EndComp
 $Comp
-L C C2
+L C-RESCUE-cryptostick C2
 U 1 1 4E2CD2C4
 P 2050 3750
@@
 $EndComp
 $Comp
-L C C1
+L C-RESCUE-cryptostick C1
 U 1 1 4E2CD2B1
 P 2050 3150
@@
 D-_PLUG
 $Comp
-L GND #PWR25
+L GND-RESCUE-cryptostick #PWR25
 U 1 1 4E2CCCBB
 P 7250 4150
@@
 $EndComp
 $Comp
-L GND #PWR28
+L GND-RESCUE-cryptostick #PWR28
 U 1 1 4E2CCC8D
 P 9850 4550
@@
 BOOT0
 $Comp
-L R R4
+L R-RESCUE-cryptostick R4
 U 1 1 530CE60F
 P 6700 5750
@@
 $EndComp
 $Comp
-L GND #PWR24
+L GND-RESCUE-cryptostick #PWR24
 U 1 1 530CE9BD
 P 7100 5800
@@
 $EndComp
 Connection ~ 6450 5450
+$Comp
+L TEST_1P W1
+U 1 1 5A282959
+P 8800 5500
+F 0 "W1" H 8800 5770 50  0000 C CNN
+F 1 "TEST_1P" H 8800 5700 50  0000 C CNN
+F 2 "SMD_Packages:1Pin" H 9000 5500 50  0001 C CNN
+F 3 "" H 9000 5500 50  0000 C CNN
+	1    8800 5500
+	1    0    0    -1
+$EndComp
+$Comp
+L TEST_1P W2
+U 1 1 5A282E6C
+P 9150 5500
+F 0 "W2" H 9150 5770 50  0000 C CNN
+F 1 "TEST_1P" H 9150 5700 50  0000 C CNN
+F 2 "SMD_Packages:1Pin" H 9350 5500 50  0001 C CNN
+F 3 "" H 9350 5500 50  0000 C CNN
+	1    9150 5500
+	1    0    0    -1
+$EndComp
+$Comp
+L TEST_1P W3
+U 1 1 5A282FD2
+P 9500 5500
+F 0 "W3" H 9500 5770 50  0000 C CNN
+F 1 "TEST_1P" H 9500 5700 50  0000 C CNN
+F 2 "SMD_Packages:1Pin" H 9700 5500 50  0001 C CNN
+F 3 "" H 9700 5500 50  0000 C CNN
+	1    9500 5500
+	1    0    0    -1
+$EndComp
+$Comp
+L TEST_1P W4
+U 1 1 5A28303D
+P 9850 5500
+F 0 "W4" H 9850 5770 50  0000 C CNN
+F 1 "TEST_1P" H 9850 5700 50  0000 C CNN
+F 2 "SMD_Packages:1Pin" H 10050 5500 50  0001 C CNN
+F 3 "" H 10050 5500 50  0000 C CNN
+	1    9850 5500
+	1    0    0    -1
+$EndComp
+Text Label 9150 5500 3    60   ~ 0
+D+_PLUG
+Text Label 9500 5500 3    60   ~ 0
+D-_PLUG
+$Comp
+L GND-RESCUE-cryptostick #PWR?
+U 1 1 5A2836B7
+P 9850 5500
+F 0 "#PWR?" H 9850 5500 30  0001 C CNN
+F 1 "GND" H 9850 5430 30  0001 C CNN
+F 2 "" H 9850 5500 60  0001 C CNN
+F 3 "" H 9850 5500 60  0001 C CNN
+	1    9850 5500
+	1    0    0    -1
+$EndComp
+Text Label 8800 5500 3    60   ~ 0
+VBUS
 $EndSCHEMATC

Commit message: DRC errors have been fixed on the original design:
- gnd power source has been added
- conflicted pin types changed to bidirectional
Connections:
- wire segments 133 -> 134
- no-connect marks 0 -> 12
Changed lines of the file:
@@
 $EndComp
 $Comp
-L GND-RESCUE-cryptostick #PWR7
+L GND-RESCUE-cryptostick #PWR01
 U 1 1 500508DE
 P 2750 1250
-F 0 "#PWR7" H 2750 1250 30  0001 C CNN
+F 0 "#PWR01" H 2750 1250 30  0001 C CNN
 F 1 "GND" H 2750 1180 30  0001 C CNN
 F 2 "" H 2750 1250 60  0001 C CNN
@@
 $EndComp
 $Comp
-L GND-RESCUE-cryptostick #PWR1
+L GND-RESCUE-cryptostick #PWR02
 U 1 1 5005072E
 P 1600 1700
-F 0 "#PWR1" H 1600 1700 30  0001 C CNN
+F 0 "#PWR02" H 1600 1700 30  0001 C CNN
 F 1 "GND" H 1600 1630 30  0001 C CNN
 F 2 "" H 1600 1700 60  0001 C CNN
@@
 $EndComp
 $Comp
-L SIM_JACKET J1
-U 1 1 500506A8
-P 2600 1650
-F 0 "J1" H 2600 1550 60  0000 C CNN
-F 1 "SIM_JACKET" H 2600 1400 60  0000 C CNN
-F 2 "" H 2600 1650 60  0001 C CNN
-F 3 "" H 2600 1650 60  0001 C CNN
-	1    2600 1650
-	1    0    0    -1
-$EndComp
-$Comp
-L GND-RESCUE-cryptostick #PWR11
+L GND-RESCUE-cryptostick #PWR03
 U 1 1 4F801E27
 P 4400 7150
-F 0 "#PWR11" H 4400 7150 30  0001 C CNN
+F 0 "#PWR03" H 4400 7150 30  0001 C CNN
 F 1 "GND" H 4400 7080 30  0001 C CNN
 F 2 "" H 4400 7150 60  0001 C CNN
@@
 $EndComp
 $Comp
-L GND-RESCUE-cryptostick #PWR14
+L GND-RESCUE-cryptostick #PWR04
 U 1 1 4F4EDF5A
 P 5150 1950
-F 0 "#PWR14" H 5150 1950 30  0001 C CNN
+F 0 "#PWR04" H 5150 1950 30  0001 C CNN
 F 1 "GND" H 5150 1880 30  0001 C CNN
 F 2 "" H 5150 1950 60  0001 C CNN
@@
 $EndComp
 $Comp
-L +3,3V #PWR12
+L +3,3V #PWR05
 U 1 1 4F4EDE58
 P 4850 1500
-F 0 "#PWR12" H 4850 1460 30  0001 C CNN
+F 0 "#PWR05" H 4850 1460 30  0001 C CNN
 F 1 "+3,3V" H 4850 1610 30  0000 C CNN
 F 2 "" H 4850 1500 60  0001 C CNN
@@
 $EndComp
 $Comp
-L GND-RESCUE-cryptostick #PWR4
+L GND-RESCUE-cryptostick #PWR06
 U 1 1 4E82CDD0
 P 1850 3600
-F 0 "#PWR4" H 1850 3600 30  0001 C CNN
+F 0 "#PWR06" H 1850 3600 30  0001 C CNN
 F 1 "GND" H 1850 3530 30  0001 C CNN
 F 2 "" H 1850 3600 60  0001 C CNN
@@
 $EndComp
 $Comp
-L GND-RESCUE-cryptostick #PWR13
+L GND-RESCUE-cryptostick #PWR07
 U 1 1 4E2D76FE
 P 4850 6100
-F 0 "#PWR13" H 4850 6100 30  0001 C CNN
+F 0 "#PWR07" H 4850 6100 30  0001 C CNN
 F 1 "GND" H 4850 6030 30  0001 C CNN
 F 2 "" H 4850 6100 60  0001 C CNN
@@
 $EndComp
 $Comp
-L GND-RESCUE-cryptostick #PWR15
+L GND-RESCUE-cryptostick #PWR08
 U 1 1 4E2D6DF1
 P 5300 6400
-F 0 "#PWR15" H 5300 6400 30  0001 C CNN
+F 0 "#PWR08" H 5300 6400 30  0001 C CNN
 F 1 "GND" H 5300 6330 30  0001 C CNN
 F 2 "" H 5300 6400 60  0001 C CNN
@@
 $EndComp
 $Comp
-L GND-RESCUE-cryptostick #PWR5
+L GND-RESCUE-cryptostick #PWR09
 U 1 1 4E2D6A81
 P 2600 4700
-F 0 "#PWR5" H 2600 4700 30  0001 C CNN
+F 0 "#PWR09" H 2600 4700 30  0001 C CNN
 F 1 "GND" H 2600 4630 30  0001 C CNN
 F 2 "" H 2600 4700 60  0001 C CNN
@@
 $EndComp
 $Comp
-L +3,3V #PWR17
+L +3,3V #PWR010
 U 1 1 4E2D6574
 P 5850 4500
-F 0 "#PWR17" H 5850 4460 30  0001 C CNN
+F 0 "#PWR010" H 5850 4460 30  0001 C CNN
 F 1 "+3,3V" H 5850 4610 30  0000 C CNN
 F 2 "" H 5850 4500 60  0001 C CNN
@@
 $EndComp
 $Comp
-L GND-RESCUE-cryptostick #PWR18
+L GND-RESCUE-cryptostick #PWR011
 U 1 1 4E2D6572
 P 5850 5100
-F 0 "#PWR18" H 5850 5100 30  0001 C CNN
+F 0 "#PWR011" H 5850 5100 30  0001 C CNN
 F 1 "GND" H 5850 5030 30  0001 C CNN
 F 2 "" H 5850 5100 60  0001 C CNN
@@
 $EndComp
 $Comp
-L +3,3V #PWR6
+L +3,3V #PWR012
 U 1 1 4E2D63FA
 P 2700 4050
-F 0 "#PWR6" H 2700 4010 30  0001 C CNN
+F 0 "#PWR012" H 2700 4010 30  0001 C CNN
 F 1 "+3,3V" H 2700 4160 30  0000 C CNN
 F 2 "" H 2700 4050 60  0001 C CNN
@@
 $EndComp
 $Comp
-L GND-RESCUE-cryptostick #PWR9
+L GND-RESCUE-cryptostick #PWR013
 U 1 1 4E2D63F8
 P 3100 3800
-F 0 "#PWR9" H 3100 3800 30  0001 C CNN
+F 0 "#PWR013" H 3100 3800 30  0001 C CNN
 F 1 "GND" H 3100 3730 30  0001 C CNN
 F 2 "" H 3100 3800 60  0001 C CNN
@@
 $EndComp
 $Comp
-L +3,3V #PWR10
+L +3,3V #PWR014
 U 1 1 4E2D167C
 P 3350 3050
-F 0 "#PWR10" H 3350 3010 30  0001 C CNN
+F 0 "#PWR014" H 3350 3010 30  0001 C CNN
 F 1 "+3,3V" H 3350 3160 30  0000 C CNN
 F 2 "" H 3350 3050 60  0001 C CNN
@@
 $EndComp
 $Comp
-L GND-RESCUE-cryptostick #PWR8
+L GND-RESCUE-cryptostick #PWR015
 U 1 1 4E2D167A
 P 2850 3200
-F 0 "#PWR8" H 2850 3200 30  0001 C CNN
+F 0 "#PWR015" H 2850 3200 30  0001 C CNN
 F 1 "GND" H 2850 3130 30  0001 C CNN
 F 2 "" H 2850 3200 60  0001 C CNN
@@
 $EndComp
 $Comp
-L GND-RESCUE-cryptostick #PWR20
+L GND-RESCUE-cryptostick #PWR016
 U 1 1 4E2D1452
 P 6450 3300
-F 0 "#PWR20" H 6450 3300 30  0001 C CNN
+F 0 "#PWR016" H 6450 3300 30  0001 C CNN
 F 1 "GND" H 6450 3230 30  0001 C CNN
 F 2 "" H 6450 3300 60  0001 C CNN
@@
 $EndComp
 $Comp
-L +3,3V #PWR16
+L +3,3V #PWR017
 U 1 1 4E2D124C
 P 5850 3050
-F 0 "#PWR16" H 5850 3010 30  0001 C CNN
+F 0 "#PWR017" H 5850 3010 30  0001 C CNN
 F 1 "+3,3V" H 5850 3160 30  0000 C CNN
 F 2 "" H 5850 3050 60  0001 C CNN
@@
 $EndComp
 $Comp
-L GND-RESCUE-cryptostick #PWR26
+L GND-RESCUE-cryptostick #PWR018
 U 1 1 4E2CDAFB
 P 7350 2950
-F 0 "#PWR26" H 7350 2950 30  0001 C CNN
+F 0 "#PWR018" H 7350 2950 30  0001 C CNN
 F 1 "GND" H 7350 2880 30  0001 C CNN
 F 2 "" H 7350 2950 60  0001 C CNN
@@
 $EndComp
 $Comp
-L +3,3V #PWR19
+L +3,3V #PWR019
 U 1 1 4E2CD995
 P 6450 1300
-F 0 "#PWR19" H 6450 1260 30  0001 C CNN
+F 0 "#PWR019" H 6450 1260 30  0001 C CNN
 F 1 "+3,3V" H 6450 1410 30  0000 C CNN
 F 2 "" H 6450 1300 60  0001 C CNN
@@
 $EndComp
 $Comp
-L GND-RESCUE-cryptostick #PWR21
+L GND-RESCUE-cryptostick #PWR020
 U 1 1 4E2CD951
 P 6600 1850
-F 0 "#PWR21" H 6600 1850 30  0001 C CNN
+F 0 "#PWR020" H 6600 1850 30  0001 C CNN
 F 1 "GND" H 6600 1780 30  0001 C CNN
 F 2 "" H 6600 1850 60  0001 C CNN
@@
 $EndComp
 $Comp
-L GND-RESCUE-cryptostick #PWR27
+L GND-RESCUE-cryptostick #PWR021
 U 1 1 4E2CD945
 P 7550 1550
-F 0 "#PWR27" H 7550 1550 30  0001 C CNN
+F 0 "#PWR021" H 7550 1550 30  0001 C CNN
 F 1 "GND" H 7550 1480 30  0001 C CNN
 F 2 "" H 7550 1550 60  0001 C CNN
@@
 $EndComp
 $Comp
-L GND-RESCUE-cryptostick #PWR22
+L GND-RESCUE-cryptostick #PWR022
 U 1 1 4E2CD8F1
 P 7050 2650
-F 0 "#PWR22" H 7050 2650 30  0001 C CNN
+F 0 "#PWR022" H 7050 2650 30  0001 C CNN
 F 1 "GND" H 7050 2580 30  0001 C CNN
 F 2 "" H 7050 2650 60  0001 C CNN
@@
 $EndComp
 $Comp
-L GND-RESCUE-cryptostick #PWR3
+L GND-RESCUE-cryptostick #PWR023
 U 1 1 4E2CD35B
 P 1775 3900
-F 0 "#PWR3" H 1775 3900 30  0001 C CNN
+F 0 "#PWR023" H 1775 3900 30  0001 C CNN
 F 1 "GND" H 1775 3830 30  0001 C CNN
 F 2 "" H 1775 3900 60  0001 C CNN
@@
 $EndComp
 $Comp
-L GND-RESCUE-cryptostick #PWR2
+L GND-RESCUE-cryptostick #PWR024
 U 1 1 4E2CD351
 P 1775 3300
-F 0 "#PWR2" H 1775 3300 30  0001 C CNN
+F 0 "#PWR024" H 1775 3300 30  0001 C CNN
 F 1 "GND" H 1775 3230 30  0001 C CNN
 F 2 "" H 1775 3300 60  0001 C CNN
@@
 D-_PLUG
 $Comp
-L GND-RESCUE-cryptostick #PWR25
+L GND-RESCUE-cryptostick #PWR025
 U 1 1 4E2CCCBB
 P 7250 4150
-F 0 "#PWR25" H 7250 4150 30  0001 C CNN
+F 0 "#PWR025" H 7250 4150 30  0001 C CNN
 F 1 "GND" H 7250 4080 30  0001 C CNN
 F 2 "" H 7250 4150 60  0001 C CNN
@@
 $EndComp
 $Comp
-L GND-RESCUE-cryptostick #PWR28
+L GND-RESCUE-cryptostick #PWR026
 U 1 1 4E2CCC8D
 P 9850 4550
-F 0 "#PWR28" H 9850 4550 30  0001 C CNN
+F 0 "#PWR026" H 9850 4550 30  0001 C CNN
 F 1 "GND" H 9850 4480 30  0001 C CNN
 F 2 "" H 9850 4550 60  0001 C CNN
@@
 	7100 5750 7100 5800
 $Comp
-L +3,3V #PWR23
+L +3,3V #PWR027
 U 1 1 530CE9AE
 P 7100 5450
-F 0 "#PWR23" H 7100 5410 30  0001 C CNN
+F 0 "#PWR027" H 7100 5410 30  0001 C CNN
 F 1 "+3,3V" H 7100 5560 30  0000 C CNN
 F 2 "" H 7100 5450 60  0000 C CNN
@@
 $EndComp
 $Comp
-L GND-RESCUE-cryptostick #PWR24
+L GND-RESCUE-cryptostick #PWR028
 U 1 1 530CE9BD
 P 7100 5800
-F 0 "#PWR24" H 7100 5800 30  0001 C CNN
+F 0 "#PWR028" H 7100 5800 30  0001 C CNN
 F 1 "GND" H 7100 5730 30  0001 C CNN
 F 2 "" H 7100 5800 60  0000 C CNN
@@
 D-_PLUG
 $Comp
-L GND-RESCUE-cryptostick #PWR?
+L GND-RESCUE-cryptostick #PWR029
 U 1 1 5A2836B7
 P 9850 5500
-F 0 "#PWR?" H 9850 5500 30  0001 C CNN
+F 0 "#PWR029" H 9850 5500 30  0001 C CNN
 F 1 "GND" H 9850 5430 30  0001 C CNN
 F 2 "" H 9850 5500 60  0001 C CNN
@@
 Text Label 8800 5500 3    60   ~ 0
 VBUS
+NoConn ~ 4800 4950
+NoConn ~ 4500 4950
+NoConn ~ 4400 4950
+NoConn ~ 4300 4950
+NoConn ~ 4200 4950
+NoConn ~ 3350 4000
+NoConn ~ 3350 3900
+NoConn ~ 3350 4100
+NoConn ~ 4400 2450
+NoConn ~ 1900 1600
+NoConn ~ 1900 1800
+NoConn ~ 3250 1800
+$Comp
+L SIM_JACKET J1
+U 1 1 500506A8
+P 2600 1650
+F 0 "J1" H 2600 1550 60  0000 C CNN
+F 1 "SIM_JACKET" H 2600 1400 60  0000 C CNN
+F 2 "" H 2600 1650 60  0001 C CNN
+F 3 "" H 2600 1650 60  0001 C CNN
+	1    2600 1650
+	1    0    0    -1
+$EndComp
+Wire Wire Line
+	9850 5500 9850 5500
+$Comp
+L PWR_FLAG #FLG030
+U 1 1 5AC017BA
+P 8000 6200
+F 0 "#FLG030" H 8000 6275 50  0001 C CNN
+F 1 "PWR_FLAG" H 8000 6350 50  0000 C CNN
+F 2 "" H 8000 6200 50  0001 C CNN
+F 3 "" H 8000 6200 50  0001 C CNN
+	1    8000 6200
+	1    0    0    -1
+$EndComp
+$Comp
+L GND-RESCUE-cryptostick #PWR031
+U 1 1 5AC01A2C
+P 8000 6200
+F 0 "#PWR031" H 8000 6200 30  0001 C CNN
+F 1 "GND" H 8000 6130 30  0001 C CNN
+F 2 "" H 8000 6200 60  0001 C CNN
+F 3 "" H 8000 6200 60  0001 C CNN
+	1    8000 6200
+	1    0    0    -1
+$EndComp
 $EndSCHEMATC

Commit message: V2
- ESD protcetion IC changed from NUF221W1 to DF5A5.6JE
- USB terminating and enable resistors have been added
- USB connector footprint has been corrected
- Many duplicated footrpints and tracks have been deleted
- GND plane on TOP side mistakenly wasnt connected to GND net.
Corrected.
- Fabrication files have been updated
- JP1 DFU selector jumper has been deleted
Parts:
- removed JP1: JUMPER, ~, symbol JUMPER
- removed U3: NUF2221W1, symbol NUF2221W1
- removed W1, W2, W3, W4: TEST_1P, SMD_Packages:1Pin, symbol TEST_1P
- added R5, R6: 22, r_0402, symbol R-RESCUE-cryptostick
- added R7: 1.5k, r_0402, symbol R-RESCUE-cryptostick
- added U3: DF5A5.6JE, TO_SOT_Packages_SMD:SOT-553, symbol DF5A5.6JE
- added p1, p2, p3, p5, p6: debug-pin, footprints:Prog_Pad_Circular, symbol debug-pin
- added p4: PROG_VCC, footprints:Prog_Pad_Circular, symbol debug-pin
- C1, C10, C11, C2, C3, C4, C5, C6, C7, C8, C9: footprint (none) -> c_0402
- D1: footprint (none) -> KPHBM-2012SURKCGKC
- J1: footprint (none) -> molex 78646-3001
- J2: footprint (none) -> USB-A-PLUG
- P1: footprint (none) -> SIL-2-2-drilled-offset
- R1, R2, R3: footprint (none) -> r_0402
- R4: footprint ~ -> r_0402
- U1: footprint (none) -> QFN36
- U2: footprint (none) -> TSOT23-5
- X1: footprint (none) -> ABM8G
Connections:
- net labels added: GND-RESCUE-cryptostick
- wire segments 134 -> 143
- no-connect marks 12 -> 13
Other:
- moved on the sheet: J2, R4

Commit message: Modifications for pro rev4 with BGA
Parts:
- added FID1, FID2: Fiducial, Fiducial:Fiducial_0.75mm_Mask1.5mm, symbol Mechanical:Fiducial
- added TP1: TestPoint, TestPoint:TestPoint_Pad_D1.5mm, symbol Connector:TestPoint
- added U1: STM32F103RBHx, Package_BGA:TFBGA-64_5x5mm_Layout8x8_P0.5mm, symbol MCU_ST_STM32F1:STM32F103RBHx
- C1, C10, C2, C3, C4, C5, C6, C7, C8: footprint c_0402 -> Capacitor_SMD:C_0402_1005Metric; symbol C-RESCUE-cryptostick -> cryptostick-rescue:C-RESCUE-cryptostick
- C11, C9: footprint c_0402 -> Capacitor_SMD:C_0402_1005Metric; symbol CP1-RESCUE-cryptostick -> cryptostick-rescue:CP1-RESCUE-cryptostick
- D1: symbol DUAL_LED -> cryptostick-rescue:DUAL_LED
- J1: symbol SIM_JACKET -> cryptostick-rescue:SIM_JACKET
- J2: symbol USB_2 -> cryptostick-rescue:USB_2
- P1: symbol CONN_4 -> cryptostick-rescue:CONN_4
- R1, R2, R3, R4, R5, R6, R7: footprint r_0402 -> Resistor_SMD:R_0402_1005Metric; symbol R-RESCUE-cryptostick -> cryptostick-rescue:R-RESCUE-cryptostick
- U2: footprint TSOT23-5 -> Package_TO_SOT_SMD:TSOT-23-5; symbol CAT6217-330 -> cryptostick-rescue:CAT6217-330
- U3: footprint TO_SOT_Packages_SMD:SOT-553 -> Package_TO_SOT_SMD:SOT-553; symbol DF5A5.6JE -> cryptostick-rescue:DF5A5.6JE
- U4: renamed from U1; footprint QFN36 -> (none); symbol STM32F103TB -> cryptostick-rescue:STM32F103TB
- X1: symbol CRYSTAL -> cryptostick-rescue:CRYSTAL
- p1, p2, p3, p4, p5, p6: symbol debug-pin -> cryptostick-rescue:debug-pin
Connections:
- net +3.3V: now also TP1.1, U1.D2 (VDD), U1.E3 (PC0), U1.E4 (VDD), U1.E5 (VDD), U1.E6 (VDD), U1.E7 (PC7), U1.E8 (PC8), U1.G1 (VREF+), U1.H1 (VDDA)
- net BOOT0: now also U1.A3 (PB9), U1.B4 (BOOT0)
- net BOOT1: now also U1.G6 (PB2), U1.H6 (PC5)
- net D+: now also U1.B8 (PA12)
- net D-: now also U1.C8 (PA11)
- net GND: now also U1.B1 (PC15), U1.C2 (VSS), U1.C3 (PB7), U1.D4 (VSS), U1.D5 (VSS), U1.D6 (VSS), U1.F1 (VSSA)
- net NRST: now also U1.E1 (NRST)
- net OSC_IN: now also U1.C1 (PD0)
- net OSC_OUT: now also U1.D1 (PD1)
- net SCCLK: now also U1.H8 (PB12)
- net SCRST: now also U1.A5 (PB3)
- net SCSDA: now also U1.G7 (PB10), U1.G8 (PB13)
- net SCVCC: now also U1.A4 (PB4), U1.B5 (PD2)
- net SWCLK: now also U1.A7 (PA14)
- net SWDIO: now also U1.A8 (PA13)
- net USB_EN: now also U1.A6 (PA15)
- net LED1: now reaches R1.2, U4.14 (PA7)
- net LED1: now also U1.H4 (PA7)
- net LED2: now reaches R2.2, U4.15 (PB0)
- net LED2: now also U1.H3 (PA4)
- no-connect marks 13 -> 14
Other:
- moved on the sheet: C1, C10, C11, C2, C3, C4, C5, C6, C7, C8, C9, D1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
