File: panel/panel-frame.kicad_pcb (KiCad board)
At the start: 2 copper layers, 107.1 x 426.9 mm, 6 parts

Commit message: Add Rev7 (BGA with smartcard pullup), update production files and panelization script.
Parts:
- added REF**: NPTH, NPTH, F.Cu at (56.5, 424.3)
- added REF**: NPTH, NPTH, F.Cu at (50.5, 2.58)
Other:
- net class Default removed
